File: layout/nfc2bid/nfc2bid.sch (KiCad schematic (older format))
At the start: 1 part, among them IC1 ARDUPROMINI

Commit message: Layoutentwurf
Signed-off-by: Claus Zielke <info@cszielke.de>
Parts:
- added D1: LED, LED_THT:LED_D3.0mm_Clear, symbol Device:LED
- added J1: Conn_01x04, Connector_PinHeader_2.54mm:PinHeader_1x04_P2.54mm_Horizontal, symbol Connector_Generic:Conn_01x04
- added R1: R, Resistor_THT:R_Axial_DIN0309_L9.0mm_D3.2mm_P12.70mm_Horizontal, symbol Device:R
- added U1: MFRC522, Zielke:MFRC522, symbol cz_module:MFRC522
- IC1: footprint (none) -> Zielke:ArduProMini
Connections:
- net GND: now reaches IC1.10 (GND)
- net GND: now also IC1.20 (GND), D1.1 (K), J1.4 (Pin_4), U1.6 (GND)
- net D9: now reaches IC1.18 (D9)
- net D9: now also U1.7 (Reset)
- net +5V: now reaches IC1.19 (RAW)
- net +5V: now also J1.1 (Pin_1)
- net VCC: now reaches IC1.22 (Vcc)
- net VCC: now also U1.8 (VCC)
- net A1: now reaches IC1.25 (A1)
- net A1: now also R1.1
- net D13: now reaches IC1.27 (D13)
- net D13: now also U1.2 (SCK)
- net D12: now reaches IC1.28 (D12)
- net D12: now also U1.4 (MISO/SCL/TX)
- net D11: now reaches IC1.29 (D11)
- net D11: now also U1.3 (MOSI)
- net D10: now reaches IC1.30 (D10)
- net D10: now also U1.1 (SS/SDA/RX)
- net SDA: now reaches IC1.31 (A4)
- net SDA: now also J1.3 (Pin_3)
- net SCL: now reaches IC1.32 (A5)
- net SCL: now also J1.2 (Pin_2)
- new net: D1.2 (A), R1.2
- no-connect marks 0 -> 17
Other:
- note added: "Grün"
- note added: "Orange"
- note added: "Schwarz"
- note added: "Weiß"
- moved on the sheet: IC1
